Commit message: set mimic joint

File: urdf/hand_v3_model_dae.urdf (robot description, URDF)
Before this commit: robot hand_v3_model, 29 links, 28 joints
Joints:
- joint index_joint1: mimic (none) -> joint=index_pulley_joint multiplier=-1.0 offset=1.0472
- joint index_joint2: mimic (none) -> joint=index_pulley_joint multiplier=-1.0 offset=1.0472
- joint index_joint3: mimic (none) -> joint=index_pulley_joint multiplier=-1.0 offset=1.0472
- joint little_joint1: mimic (none) -> joint=little_pulley_joint multiplier=1.0 offset=1.0472
- joint little_joint2: mimic (none) -> joint=little_pulley_joint multiplier=1.0 offset=1.0472
- joint little_joint3: mimic (none) -> joint=little_pulley_joint multiplier=1.0 offset=1.0472
- joint middle_joint1: mimic (none) -> joint=middle_pulley_joint multiplier=1.0 offset=0.87267
- joint middle_joint2: mimic (none) -> joint=middle_pulley_joint multiplier=1.0 offset=0.87267
- joint middle_joint3: mimic (none) -> joint=middle_pulley_joint multiplier=1.0 offset=0.87267
- joint ring_joint1: mimic (none) -> joint=ring_pulley_joint multiplier=-1.0 offset=1.0472
- joint ring_joint2: mimic (none) -> joint=ring_pulley_joint multiplier=-1.0 offset=1.0472
- joint ring_joint3: mimic (none) -> joint=ring_pulley_joint multiplier=-1.0 offset=1.0472
- joint thumb_joint1: mimic (none) -> joint=thumb_pulley_joint multiplier=1.0 offset=1.0472
- joint thumb_joint2: mimic (none) -> joint=thumb_pulley_joint multiplier=1.0 offset=1.0472

Commit message: update

File: urdf/hand_v3_model_dae.urdf (robot description, URDF)
Before this commit: robot hand_v3_model, 30 links, 29 joints
Joints:
- joint arm_joint0: limit lower=-2.06167 upper=0.41233 effort=0.0 velocity=4.553 -> lower=-2.3562 upper=2.3562 effort=0.0 velocity=4.553
- joint arm_joint2: limit lower=-1.5708 upper=0.06 effort=0.0 velocity=6.545 -> lower=-2.3562 upper=2.3562 effort=0.0 velocity=6.545
- joint hand_base_joint: limit lower=-1.5708 upper=1.5708 effort=0.0 velocity=6.545 -> lower=-2.3562 upper=2.3562 effort=0.0 velocity=6.545
